Commit message: New version of controller, test framework and multiple testscenarios

File: ws/src/magnetic_controller/robots/simple_robot.urdf (robot description, URDF)
Before this commit: robot simple robot, 4 links, 3 joints
Joints:
- removed joint jointX
- removed joint jointY
- removed joint jointZ
- added joint jointX_joint: type prismatic, parent link0, child link1, axis 1 0 0, limit lower=-100 upper=100 effort=1000.0 velocity=0.2
- added joint jointY_joint: type prismatic, parent link1, child link2, axis 0 1 0, limit lower=-100 upper=100 effort=1000.0 velocity=0.2
- added joint jointZ_joint: type prismatic, parent link2, child eef_link, axis 0 0 1, limit lower=-100 upper=100 effort=1000.0 velocity=0.2

Commit message: Added latest changes to controller. Also testing framework, scenarios and testbenches

File: ws/src/magnetic_controller/robots/simple_robot.urdf (robot description, URDF)
Before this commit: robot simple robot, 4 links, 3 joints
Links:
- link eef_link: geometry collision sphere radius=0.025; visual sphere radius=0.025
